File: KiCAD/didot.kicad_pcb (KiCad board)
At the start: 2 copper layers, 156.2 x 118.1 mm, 77 parts, among them J1 JST_BATTERY, J2 Display Socket, U1 nice!nano

Commit message: Whatever was on my PC
Parts:
- JP1: value VCC -> 3v3
- moved SW_PWR1 36.3 mm to (59.7, 40.1), turned to -90 degrees
- moved TH1 35.1 mm to (60.3, 66.1), turned to 90 degrees
- moved TH1 33.9 mm to (94.3, 66.1), turned to 90 degrees
- moved TH1 33.1 mm to (60.3, 33.1), turned to 90 degrees
- moved TH1 32.0 mm to (94.3, 33.1), turned to 90 degrees
- moved J2 25.4 mm to (77.3, 66.6), turned to 0 degrees
- moved JP1 19.2 mm to (61.7, 60.3), turned to 90 degrees
- moved SW_RESET1 16.5 mm to (59.7, 53.1), turned to 90 degrees
- moved JP2 15.3 mm to (64.3, 60.3), turned to 90 degrees
- moved JP3 9.33 mm to (66.9, 60.3), turned to 90 degrees
- moved JP4 7.39 mm to (69.5, 60.3), turned to 90 degrees
- moved DA5 6.45 mm to (192.5, 56.5)
- moved DB5 6.10 mm to (192.5, 73.5)
- moved DC5 5.84 mm to (192.5, 90.5)
- moved SWA5 5.77 mm to (198.0, 49.5)
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Connections:
- net VCC renamed VBAT
- net VCOM renamed 3v3
- JP1 pad 1: Net-(J2-Pad1) -> Net-(J2-Pad2)
- JP1 pad 3: Net-(J2-Pad9) -> Net-(J2-Pad8)
Routing:
- net Net-(J2-Pad9): track 21.6 -> 0.00 mm
- net col4: track 334.0 -> 314.7 mm, vias 6 -> 7
- net rowD: track 186.7 -> 168.4 mm, vias 2 -> 1
- net col3: track 304.6 -> 287.5 mm, vias 6 -> 7
- net Net-(J2-Pad3): track 16.7 -> 0.00 mm
- net Net-(J1-Pad1): track 43.8 -> 27.2 mm
- net VBAT: track 47.6 -> 31.8 mm, vias 1 -> 0
- net Net-(J2-Pad4): track 15.6 -> 0.00 mm, vias 1 -> 0
- net RESET: track 44.3 -> 29.3 mm
- net rowA: track 149.5 -> 134.8 mm, vias 2 -> 1
- net col2: track 281.5 -> 267.5 mm, vias 6 -> 7
- net rowC: track 172.4 -> 158.5 mm, vias 2 -> 1
- net rowB: track 151.7 -> 139.4 mm, vias 2 -> 1
- net Net-(U1-Pad2): track 27.9 -> 17.0 mm
- net Net-(J2-Pad6): track 10.3 -> 0.00 mm, vias 1 -> 0
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Other:
- board size 156.2 x 118.1 mm -> 156.2 x 118.2 mm
- net class Default removed
